File: beaucoup_main/beaucoup_main.kicad_pcb (KiCad board)
At the start: 2 copper layers, 21 parts, among them J1 RGBled, J10 Conn_01x03_Pin, J11 AMP, J12 tomist, J2 NFCreader, J3 potenziometro, J5 conn_bottone_mist, J6 Conn_01x02_Pin, J7 Conn_01x02_Pin, J8 Conn_01x02_Pin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

Commit message: Main pcb should be ready for production
Parts:
- added J4: Conn_01x02_Pin, Connector_PinHeader_2.54mm:PinHeader_1x02_P2.54mm_Vertical, F.Cu at (121.9, 68.5)
- moved H3 200.2 mm to (112.8, 72.1)
- moved H4 150.6 mm to (179.6, 72.1)
- moved H2 131.3 mm to (179.6, 120.6)
- moved J9 110.2 mm to (127.0, 68.5), turned to 0 degrees
- moved J7 97.7 mm to (161.2, 96.9)
- moved J8 89.5 mm to (172.0, 83.5), turned to -90 degrees
- moved H1 87.9 mm to (112.8, 120.6)
- moved J1 52.3 mm to (161.8, 74.1)
- moved J11 52.3 mm to (161.3, 112.5)
- moved J2 52.3 mm to (161.3, 89.9)
- moved J3 52.3 mm to (170.7, 70.3)
- moved J6 52.3 mm to (169.4, 96.9)
- moved Q1 52.3 mm to (128.8, 77.8)
- moved R1 52.3 mm to (129.4, 81.0)
- moved R2 52.3 mm to (129.4, 83.5)
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Connections:
- J9 pad 2: +3.3V -> +5V
Routing:
- net +3.3V: track 0.00 -> 65.7 mm, vias 0 -> 1
- net +5V: track 0.00 -> 38.5 mm, vias 0 -> 6
- net Net-(J2-Pin_5): track 0.00 -> 37.2 mm, vias 0 -> 2
- net POT: track 0.00 -> 37.1 mm
- net uRX: track 0.00 -> 28.7 mm
- net SDA: track 0.00 -> 28.6 mm
- net SCL: track 0.00 -> 25.7 mm
- net uTX: track 0.00 -> 20.5 mm
- net BTN: track 0.00 -> 19.4 mm
- net IRQ: track 0.00 -> 16.7 mm
- net Net-(J11-Pin_1): track 0.00 -> 16.3 mm
- net LEDR: track 0.00 -> 11.9 mm
- net LEDG: track 0.00 -> 11.9 mm
- net LEDB: track 0.00 -> 11.9 mm
- net Net-(J12-Pin_1): track 0.00 -> 8.24 mm
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- added copper zone on In1.Cu, net (none)
Other:
- board outline added: 79.2 x 62.7 mm
- copper layers 2 -> 4
- board text added: "Tutti i buchi sono per M3"
