File: beaucoup_rgb/beaucoup_rgb.kicad_pcb (KiCad board)
At the start: 2 copper layers, 22.2 x 12.1 mm, 6 parts, among them J1 Conn_01x04_Pin

Commit message: Aggiunge file lavorazione rgb revA
Parts:
- J1: footprint Connector_PinHeader_2.54mm:PinHeader_1x04_P2.54mm_Vertical -> Connector_JST:JST_XH_B4B-XH-A_1x04_P2.50mm_Vertical
- turned J1 to 0 degrees
Changed lines of the file:
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@@
     )
   )
-  (footprint "Connector_PinHeader_2.54mm:PinHeader_1x04_P2.54mm_Vertical" (layer "F.Cu")
-    (at 157.48 101.6 90)
-    (descr "Through hole straight pin header, 1x04, 2.54mm pitch, single row")
-    (tags "Through hole pin header THT 1x04 2.54mm single row")
+  (footprint "Connector_JST:JST_XH_B4B-XH-A_1x04_P2.50mm_Vertical" (layer "F.Cu")
+    (at 157.48 101.6)
+    (descr "JST XH series connector, B4B-XH-A (http://www.jst-mfg.com/product/pdf/eng/eXH.pdf), generated with kicad-footprint-generator")
+    (tags "connector JST XH vertical")
     (property "Sheetfile" "beaucoup_rgb.kicad_sch")
     (property "Sheetname" "")
@@
     (property "ki_keywords" "connector")
     (attr through_hole)
-    (fp_text reference "J1" (at 0 -2.33 90) (layer "F.SilkS")
-        (effects (font (size 1 1) (thickness 0.15)))
-    )
-    (fp_text value "Conn_01x04_Pin" (at 1.27 9.95 90) (layer "F.Fab")
-        (effects (font (size 1 1) (thickness 0.15)))
-    )
-    (fp_text user "${REFERENCE}" (at 0 3.81) (layer "F.Fab")
-        (effects (font (size 1 1) (thickness 0.15)))
-    )
-    (fp_line (start -1.33 -1.33) (end 0 -1.33)
-      (stroke (width 0.12) (type solid)) (layer "F.SilkS"))
-    (fp_line (start -1.33 0) (end -1.33 -1.33)
-      (stroke (width 0.12) (type solid)) (layer "F.SilkS"))
-    (fp_line (start -1.33 1.27) (end -1.33 8.95)
-      (stroke (width 0.12) (type solid)) (layer "F.SilkS"))
-    (fp_line (start -1.33 1.27) (end 1.33 1.27)
-      (stroke (width 0.12) (type solid)) (layer "F.SilkS"))
-    (fp_line (start -1.33 8.95) (end 1.33 8.95)
-      (stroke (width 0.12) (type solid)) (layer "F.SilkS"))
-    (fp_line (start 1.33 1.27) (end 1.33 8.95)
-      (stroke (width 0.12) (type solid)) (layer "F.SilkS"))
-    (fp_line (start -1.8 -1.8) (end -1.8 9.4)
-      (stroke (width 0.05) (type solid)) (layer "F.CrtYd"))
-    (fp_line (start -1.8 9.4) (end 1.8 9.4)
-      (stroke (width 0.05) (type solid)) (layer "F.CrtYd"))
-    (fp_line (start 1.8 -1.8) (end -1.8 -1.8)
-      (stroke (width 0.05) (type solid)) (layer "F.CrtYd"))
-    (fp_line (start 1.8 9.4) (end 1.8 -1.8)
-      (stroke (width 0.05) (type solid)) (layer "F.CrtYd"))
-    (fp_line (start -1.27 -0.635) (end -0.635 -1.27)
-      (stroke (width 0.1) (type solid)) (layer "F.Fab"))
-    (fp_line (start -1.27 8.89) (end -1.27 -0.635)
-      (stroke (width 0.1) (type solid)) (layer "F.Fab"))
-    (fp_line (start -0.635 -1.27) (end 1.27 -1.27)
-      (stroke (width 0.1) (type solid)) (layer "F.Fab"))
-    (fp_line (start 1.27 -1.27) (end 1.27 8.89)
-      (stroke (width 0.1) (type solid)) (layer "F.Fab"))
-    (fp_line (start 1.27 8.89) (end -1.27 8.89)
-      (stroke (width 0.1) (type solid)) (layer "F.Fab"))
-    (pad "1" thru_hole rect (at 0 0 90) (size 1.7 1.7) (drill 1) (layers "*.Cu" "*.Mask")
+    (fp_text reference "J1" (at 3.75 -3.55) (layer "F.SilkS")
+        (effects (font (size 1 1) (thickness 0.15)))
+    )
+    (fp_text value "Conn_01x04_Pin" (at 3.75 4.6) (layer "F.Fab")
+        (effects (font (size 1 1) (thickness 0.15)))
+    )
+    (fp_text user "${REFERENCE}" (at 3.75 2.7) (layer "F.Fab")
+        (effects (font (size 1 1) (thickness 0.15)))
+    )
+    (fp_line (start -2.85 -2.75) (end -2.85 -1.5)
+      (stroke (width 0.12) (type solid)) (layer "F.SilkS"))
+    (fp_line (start -2.56 -2.46) (end -2.56 3.51)
+      (stroke (width 0.12) (type solid)) (layer "F.SilkS"))
+    (fp_line (start -2.56 3.51) (end 10.06 3.51)
+      (stroke (width 0.12) (type solid)) (layer "F.SilkS"))
+    (fp_line (start -2.55 -2.45) (end -2.55 -1.7)
+      (stroke (width 0.12) (type solid)) (layer "F.SilkS"))
+    (fp_line (start -2.55 -1.7) (end -0.75 -1.7)
+      (stroke (width 0.12) (type solid)) (layer "F.SilkS"))
+    (fp_line (start -2.55 -0.2) (end -1.8 -0.2)
+      (stroke (width 0.12) (type solid)) (layer "F.SilkS"))
+    (fp_line (start -1.8 -0.2) (end -1.8 2.75)
+      (stroke (width 0.12) (type solid)) (layer "F.SilkS"))
+    (fp_line (start -1.8 2.75) (end 3.75 2.75)
+      (stroke (width 0.12) (type solid)) (layer "F.SilkS"))
+    (fp_line (start -1.6 -2.75) (end -2.85 -2.75)
+      (stroke (width 0.12) (type solid)) (layer "F.SilkS"))
+    (fp_line (start -0.75 -2.45) (end -2.55 -2.45)
+      (stroke (width 0.12) (type solid)) (layer "F.SilkS"))
+    (fp_line (start -0.75 -1.7) (end -0.75 -2.45)
+      (stroke (width 0.12) (type solid)) (layer "F.SilkS"))
+    (fp_line (start 0.75 -2.45) (end 0.75 -1.7)
+      (stroke (width 0.12) (type solid)) (layer "F.SilkS"))
+    (fp_line (start 0.75 -1.7) (end 6.75 -1.7)
+      (stroke (width 0.12) (type solid)) (layer "F.SilkS"))
+    (fp_line (start 6.75 -2.45) (end 0.75 -2.45)
+      (stroke (width 0.12) (type solid)) (layer "F.SilkS"))
+    (fp_line (start 6.75 -1.7) (end 6.75 -2.45)
+      (stroke (width 0.12) (type solid)) (layer "F.SilkS"))
+    (fp_line (start 8.25 -2.45) (end 8.25 -1.7)
+      (stroke (width 0.12) (type solid)) (layer "F.SilkS"))
+    (fp_line (start 8.25 -1.7) (end 10.05 -1.7)
+      (stroke (width 0.12) (type solid)) (layer "F.SilkS"))
+    (fp_line (start 9.3 -0.2) (end 9.3 2.75)
+      (stroke (width 0.12) (type solid)) (layer "F.SilkS"))
+    (fp_line (start 9.3 2.75) (end 3.75 2.75)
+      (stroke (width 0.12) (type solid)) (layer "F.SilkS"))
+    (fp_line (start 10.05 -2.45) (end 8.25 -2.45)
+      (stroke (width 0.12) (type solid)) (layer "F.SilkS"))
+    (fp_line (start 10.05 -1.7) (end 10.05 -2.45)
+      (stroke (width 0.12) (type solid)) (layer "F.SilkS"))
+    (fp_line (start 10.05 -0.2) (end 9.3 -0.2)
+      (stroke (width 0.12) (type solid)) (layer "F.SilkS"))
+    (fp_line (start 10.06 -2.46) (end -2.56 -2.46)
+      (stroke (width 0.12) (type solid)) (layer "F.SilkS"))
+    (fp_line (start 10.06 3.51) (end 10.06 -2.46)
+      (stroke (width 0.12) (type solid)) (layer "F.SilkS"))
+    (fp_line (start -2.95 -2.85) (end -2.95 3.9)
+      (stroke (width 0.05) (type solid)) (layer "F.CrtYd"))
+    (fp_line (start -2.95 3.9) (end 10.45 3.9)
+      (stroke (width 0.05) (type solid)) (layer "F.CrtYd"))
+    (fp_line (start 10.45 -2.85) (end -2.95 -2.85)
+      (stroke (width 0.05) (type solid)) (layer "F.CrtYd"))
+    (fp_line (start 10.45 3.9) (end 10.45 -2.85)
+      (stroke (width 0.05) (type solid)) (layer "F.CrtYd"))
+    (fp_line (start -2.45 -2.35) (end -2.45 3.4)
+      (stroke (width 0.1) (type solid)) (layer "F.Fab"))
+    (fp_line (start -2.45 3.4) (end 9.95 3.4)
+      (stroke (width 0.1) (type solid)) (layer "F.Fab"))
+    (fp_line (start -0.625 -2.35) (end 0 -1.35)
+      (stroke (width 0.1) (type solid)) (layer "F.Fab"))
+    (fp_line (start 0 -1.35) (end 0.625 -2.35)
+      (stroke (width 0.1) (type solid)) (layer "F.Fab"))
+    (fp_line (start 9.95 -2.35) (end -2.45 -2.35)
+      (stroke (width 0.1) (type solid)) (layer "F.Fab"))
+    (fp_line (start 9.95 3.4) (end 9.95 -2.35)
+      (stroke (width 0.1) (type solid)) (layer "F.Fab"))
+    (pad "1" thru_hole roundrect (at 0 0) (size 1.7 1.95) (drill 0.95) (layers "*.Cu" "*.Mask") (roundrect_rratio 0.147059)
       (net 5 "Net-(J1-Pin_1)") (pinfunction "Pin_1") (pintype "passive"))
-    (pad "2" thru_hole oval (at 0 2.54 90) (size 1.7 1.7) (drill 1) (layers "*.Cu" "*.Mask")
+    (pad "2" thru_hole oval (at 2.5 0) (size 1.7 1.95) (drill 0.95) (layers "*.Cu" "*.Mask")
       (net 6 "Net-(J1-Pin_2)") (pinfunction "Pin_2") (pintype "passive"))
-    (pad "3" thru_hole oval (at 0 5.08 90) (size 1.7 1.7) (drill 1) (layers "*.Cu" "*.Mask")
+    (pad "3" thru_hole oval (at 5 0) (size 1.7 1.95) (drill 0.95) (layers "*.Cu" "*.Mask")
       (net 7 "Net-(J1-Pin_3)") (pinfunction "Pin_3") (pintype "passive"))
-    (pad "4" thru_hole oval (at 0 7.62 90) (size 1.7 1.7) (drill 1) (layers "*.Cu" "*.Mask")
+    (pad "4" thru_hole oval (at 7.5 0) (size 1.7 1.95) (drill 0.95) (layers "*.Cu" "*.Mask")
       (net 2 "Net-(D1-A)") (pinfunction "Pin_4") (pintype "passive"))
-    (model "${KICAD6_3DMODEL_DIR}/Connector_PinHeader_2.54mm.3dshapes/PinHeader_1x04_P2.54mm_Vertical.wrl" hide
-      (opacity 0.2800)      (offset (xyz 0 0 0))
+    (model "${KICAD6_3DMODEL_DIR}/Connector_JST.3dshapes/JST_XH_B4B-XH-A_1x04_P2.50mm_Vertical.wrl"
+      (offset (xyz 0 0 0))
       (scale (xyz 1 1 1))
-      (rotate (xyz 180 90 0))
-    )
-    (model "${KICAD7_3DMODEL_DIR}/Connector_PinHeader_2.54mm.3dshapes/PinHeader_1x04_P2.54mm_Horizontal.wrl"
-      (offset (xyz 0 0 -1.5))
-      (scale (xyz 1 1 1))
-      (rotate (xyz 0 -180 0))
+      (rotate (xyz 0 0 0))
     )
   )
@@
       )
     )
+  )
+  (zone (net 0) (net_name "") (layer "User.3") (hatch edge 0.5)
+    (connect_pads (clearance 0.5))
+    (min_thickness 0.25) (filled_areas_thickness no)
+    (fill yes (thermal_gap 0.5) (thermal_bridge_width 0.5) (smoothing fillet) (radius 1))
+    (polygon
+      (pts
+        (xy 144.5 105.5)
+        (xy 171 105.5)
+        (xy 171 90)
+        (xy 144.5 90)
+      )
+    )
