File: beaucoup_rgb/beaucoup_rgb.kicad_sch (KiCad schematic)
At the start: 6 parts, among them J1 Conn_01x04_Pin

Commit message: Aggiunge file lavorazione rgb revA
Parts:
- J1: footprint Connector_PinHeader_2.54mm:PinHeader_1x04_P2.54mm_Vertical -> Connector_JST:JST_XH_B4B-XH-A_1x04_P2.50mm_Vertical
Changed lines of the file:
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@@
       (effects (font (size 1.27 1.27)))
     )
-    (property "Footprint" "Connector_PinHeader_2.54mm:PinHeader_1x04_P2.54mm_Vertical" (at 111.76 90.17 0)
+    (property "Footprint" "Connector_JST:JST_XH_B4B-XH-A_1x04_P2.50mm_Vertical" (at 111.76 90.17 0)
       (effects (font (size 1.27 1.27)) hide)
     )
